File: KiCad/DIY.kicad_pcb (KiCad board)
At the start: 2 copper layers, 81.3 x 62.2 mm, 24 parts, among them J1 AVR-ISP-6, SW1 red, SW2 yellow, SW3 green, SW4 blue, SW5 SW_SPST, U1 ATmega168A-P, Y1 16.00Mhz

Commit message: buzzer update
Parts:
- added G***: LOGO, Mike:portrait_35mm, B.Cu at (106.4, 111.8)
- LS1: footprint SamacSys_Parts:CPT111783SMTTR -> SamacSys_Parts:PKM13EPYH4002-B0
- R1: value 10Ω -> 120Ω
- R2: value 330Ω -> 120Ω
- R3: value 330Ω -> 220Ω
- R4: value 470Ω -> 220Ω
- moved LS1 5.39 mm to (81.1, 92.5), turned to 0 degrees
- moved SW2 0.21 mm to (138.8, 118.4)
- renumbered TEST to JP1
Routing:
- net GND: track 18.5 -> 14.3 mm, vias 1 -> 0
- net /MISO: track 56.5 -> 55.6 mm
Other:
- board text added: "Simon Game D.I.Y version 1.0"
- board text added: "https://github.com/mikeymcfish/SimonGame"
- board text removed: "SPEAKER"
