File: KiCad/DIY.kicad_sch (KiCad schematic)
At the start: 24 parts, among them J1 AVR-ISP-6, SW1 red, SW2 yellow, SW3 green, SW4 blue, SW5 SW_SPST, U1 ATmega168A-P, Y1 16.00Mhz

Commit message: buzzer update
Parts:
- LS1: footprint SamacSys_Parts:CPT111783SMTTR -> SamacSys_Parts:PKM13EPYH4002-B0
- R1: value 10Ω -> 120Ω
- R2: value 330Ω -> 120Ω
- R3: value 330Ω -> 220Ω
- R4: value 470Ω -> 220Ω
Changed lines of the file:
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@@
       (effects (font (size 1.27 1.27)) (justify left))
     )
-    (property "Value" "470Ω" (id 1) (at 116.84 147.32 90)
+    (property "Value" "220Ω" (id 1) (at 116.84 147.32 90)
       (effects (font (size 1.27 1.27)) (justify left))
     )
@@
       (effects (font (size 1.27 1.27)) (justify left))
     )
-    (property "Footprint" "SamacSys_Parts:CPT111783SMTTR" (id 2) (at 110.49 102.87 0)
+    (property "Footprint" "SamacSys_Parts:PKM13EPYH4002-B0" (id 2) (at 110.49 102.87 0)
       (effects (font (size 1.27 1.27)) hide)
     )
@@
       (effects (font (size 1.27 1.27)) (justify left))
     )
-    (property "Value" "330Ω" (id 1) (at 116.84 139.7 90)
+    (property "Value" "220Ω" (id 1) (at 116.84 139.7 90)
       (effects (font (size 1.27 1.27)) (justify left))
     )
@@
       (effects (font (size 1.27 1.27)) (justify left))
     )
-    (property "Value" "330Ω" (id 1) (at 116.84 132.08 90)
+    (property "Value" "120Ω" (id 1) (at 116.84 132.08 90)
       (effects (font (size 1.27 1.27)) (justify left))
     )
@@
     (in_bom yes) (on_board yes)
     (property "Reference" "R1" (id 0) (at 114.3 120.65 90))
-    (property "Value" "10Ω" (id 1) (at 114.3 124.46 90))
+    (property "Value" "120Ω" (id 1) (at 114.3 124.46 90))
     (property "Footprint" "Resistor_THT:R_Axial_DIN0207_L6.3mm_D2.5mm_P10.16mm_Horizontal" (id 2) (at 111.76 121.92 0)
       (effects (font (size 1.27 1.27)) hide)
@@
     )
     (path "/960cb7f4-0c08-41c0-b8ff-fa20c1cc8bf2"
-      (reference "LS1") (unit 1) (value "Speaker") (footprint "SamacSys_Parts:CPT111783SMTTR")
+      (reference "LS1") (unit 1) (value "Speaker") (footprint "SamacSys_Parts:PKM13EPYH4002-B0")
     )
     (path "/d720c83b-7eb4-437b-851d-0c48c626245f"
-      (reference "R1") (unit 1) (value "10Ω") (footprint "Resistor_THT:R_Axial_DIN0207_L6.3mm_D2.5mm_P10.16mm_Horizontal")
+      (reference "R1") (unit 1) (value "120Ω") (footprint "Resistor_THT:R_Axial_DIN0207_L6.3mm_D2.5mm_P10.16mm_Horizontal")
     )
     (path "/b50c6642-ec2d-4f21-8bcb-af36206e84ce"
-      (reference "R2") (unit 1) (value "330Ω") (footprint "Resistor_THT:R_Axial_DIN0207_L6.3mm_D2.5mm_P10.16mm_Horizontal")
+      (reference "R2") (unit 1) (value "120Ω") (footprint "Resistor_THT:R_Axial_DIN0207_L6.3mm_D2.5mm_P10.16mm_Horizontal")
     )
     (path "/a5104a57-c32b-4047-88ce-239a8e9750f5"
-      (reference "R3") (unit 1) (value "330Ω") (footprint "Resistor_THT:R_Axial_DIN0207_L6.3mm_D2.5mm_P10.16mm_Horizontal")
+      (reference "R3") (unit 1) (value "220Ω") (footprint "Resistor_THT:R_Axial_DIN0207_L6.3mm_D2.5mm_P10.16mm_Horizontal")
     )
     (path "/82d3c384-2ad1-4b86-941e-63010036e8d6"
-      (reference "R4") (unit 1) (value "470Ω") (footprint "Resistor_THT:R_Axial_DIN0207_L6.3mm_D2.5mm_P10.16mm_Horizontal")
+      (reference "R4") (unit 1) (value "220Ω") (footprint "Resistor_THT:R_Axial_DIN0207_L6.3mm_D2.5mm_P10.16mm_Horizontal")
     )
     (path "/93d0e0ea-0245-4d61-aa0f-470145544613"
@@
       (reference "SW1") (unit 1) (value "red") (footprint "Button_Switch_THT:SW_PUSH_6mm")
     )
-    (path "/fd73bab2-fc71-4b2e-9d46-53bd4b06d591"
+    (path "/fd73bab2-fc71-4b2e-9d46-53bd4b06d592"
       (reference "SW2") (unit 1) (value "yellow") (footprint "Button_Switch_THT:SW_PUSH_6mm")
     )
